File: fabrication/circuitboard/Basic-ADSR.kicad_pcb (KiCad board)
At the start: 2 copper layers, 20 x 109.5 mm, 33 parts, among them J2 Power Input, J3 Conn_Circuit, J4 Conn_Circuit, Q1 BC547, Q2 BC547, Q3 BC547, U1 TL072, U2 LM555xN

Commit message: update GND plane for circuitboard following issues
Routing:
- net GND: track 0.00 -> 9.73 mm, vias 0 -> 20
Other:
- board text added: "Basic ADSR 1.1 Bleep Sound 2024"
- board text removed: "Basic ADSR 1.0 Bleep Sound 2023"
Changed lines of the file:
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@@
     (effects (font (size 1 1) (thickness 0.15)) (justify mirror))
   )
-  (gr_text "Basic ADSR 1.0\nBleep Sound 2023" (at 38.6 122.4) (layer "F.SilkS")
+  (gr_text "Basic ADSR 1.1\nBleep Sound 2024" (at 38.6 122.4) (layer "F.SilkS")
     (effects (font (size 1 1) (thickness 0.15)))
   )
@@
     (style (thickness 0.15) (arrow_length 1.27) (text_position_mode 0) (extension_height 0.58642) (extension_offset 0.5) keep_text_aligned)
   )
+  (segment (start 43.9 64.4) (end 44.9 63.4) (width 0.25) (layer "F.Cu") (net 1))
+  (segment (start 44.9 56.5) (end 43.9 55.5) (width 0.25) (layer "F.Cu") (net 1))
+  (segment (start 44.9 63.4) (end 44.9 56.5) (width 0.25) (layer "F.Cu") (net 1))
+  (via (at 29.9495 71.2) (size 0.8) (drill 0.4) (layers "F.Cu" "B.Cu") (free) (net 1))
+  (via (at 36 45.3) (size 0.8) (drill 0.4) (layers "F.Cu" "B.Cu") (free) (net 1))
+  (via (at 43.9 64.4) (size 0.8) (drill 0.4) (layers "F.Cu" "B.Cu") (free) (net 1))
+  (via (at 46.5 68.5) (size 0.8) (drill 0.4) (layers "F.Cu" "B.Cu") (free) (net 1))
+  (via (at 40.8 40.3) (size 0.8) (drill 0.4) (layers "F.Cu" "B.Cu") (free) (net 1))
+  (via (at 30.7 70.5) (size 0.8) (drill 0.4) (layers "F.Cu" "B.Cu") (free) (net 1))
+  (via (at 43.9 55.5) (size 0.8) (drill 0.4) (layers "F.Cu" "B.Cu") (free) (net 1))
+  (via (at 33.2 97) (size 0.8) (drill 0.4) (layers "F.Cu" "B.Cu") (free) (net 1))
+  (via (at 31.4 69.7) (size 0.8) (drill 0.4) (layers "F.Cu" "B.Cu") (free) (net 1))
+  (via (at 40.6 57.5) (size 0.8) (drill 0.4) (layers "F.Cu" "B.Cu") (free) (net 1))
+  (via (at 43.9 66.4) (size 0.8) (drill 0.4) (layers "F.Cu" "B.Cu") (free) (net 1))
+  (via (at 34.1 43.9) (size 0.8) (drill 0.4) (layers "F.Cu" "B.Cu") (free) (net 1))
+  (via (at 34.2 97) (size 0.8) (drill 0.4) (layers "F.Cu" "B.Cu") (free) (net 1))
+  (via (at 43.9 65.4) (size 0.8) (drill 0.4) (layers "F.Cu" "B.Cu") (free) (net 1))
+  (via (at 46.5 69.5) (size 0.8) (drill 0.4) (layers "F.Cu" "B.Cu") (free) (net 1))
+  (via (at 39.8 40.3) (size 0.8) (drill 0.4) (layers "F.Cu" "B.Cu") (free) (net 1))
+  (via (at 40.6 58.5) (size 0.8) (drill 0.4) (layers "F.Cu" "B.Cu") (free) (net 1))
+  (via (at 36 46.2) (size 0.8) (drill 0.4) (layers "F.Cu" "B.Cu") (free) (net 1))
+  (via (at 40.3 39.3) (size 0.8) (drill 0.4) (layers "F.Cu" "B.Cu") (free) (net 1))
+  (via (at 43.9 54.5) (size 0.8) (drill 0.4) (layers "F.Cu" "B.Cu") (free) (net 1))
   (segment (start 40.8 137.9) (end 34.92 137.9) (width 0.6) (layer "F.Cu") (net 2))
   (segment (start 34.92 137.9) (end 34.8 137.78) (width 0.6) (layer "F.Cu") (net 2))
