File: fabrication/front/Basic-ADSR.kicad_pcb (KiCad board)
At the start: 2 copper layers, 20 x 128.5 mm, 2 parts

Commit message: update GND plane for circuitboard following issues
Other:
- board text added: "Basic ADSR 1.1 Bleep Sound 2024"
- board text removed: "Basic ADSR 1.0 Bleep Sound 2023"
Changed lines of the file:
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@@
   (gr_line (start 89.5 24.5) (end 109.5 24.5)
     (stroke (width 0.05) (type solid)) (layer "Edge.Cuts"))
-  (gr_text "Basic ADSR 1.0\nBleep Sound 2023" (at 99.5 32.5) (layer "B.SilkS")
+  (gr_text "Basic ADSR 1.1\nBleep Sound 2024" (at 99.5 32.5) (layer "B.SilkS")
     (effects (font (size 1 1) (thickness 0.15)) (justify mirror))
   )
